Commit message: Bachelorarbeit: gesamter selbst geschriebener Quellcode (Stand 2026-09-28)

File: quellcode/src/mycobot_world/urdf/mycobot_world.urdf.xacro (robot description, xacro)
@@ -13,14 +13,33 @@
   -->
   <xacro:property name="PI" value="3.14159265358979323846"/>
+  <!-- Kamera-Pose (cam_x/y/z, cam_roll/pitch/yaw) kommt aus EINER erzeugten Datei.
+       tools/auto_camera_calibration.py schreibt sie nach jeder Messung neu; diese Datei
+       hier bleibt dabei unberührt. Kamera UND Kamera-Arm werden daraus nachgeführt. -->
+  <xacro:include filename="$(find mycobot_world)/urdf/camera_pose.xacro"/>
+  <!-- Bereitstellungsschale: Masse in schale.xacro, Lage in schale_pose.xacro
+       (erzeugt von tools/schale_pose_klicken.py, wie camera_pose.xacro). -->
+  <xacro:include filename="$(find mycobot_world)/urdf/schale.xacro"/>
+  <xacro:include filename="$(find mycobot_world)/urdf/schale_pose.xacro"/>
+  <!-- Trichter (Vereinzelung): Masse in trichter.xacro, Lage in trichter_pose.xacro. -->
+  <xacro:include filename="$(find mycobot_world)/urdf/trichter.xacro"/>
+  <xacro:include filename="$(find mycobot_world)/urdf/trichter_pose.xacro"/>
+  <!-- Ablageplatte (5x4 Nester): Masse in ablageplatte.xacro, Lage + Bosse aus den
+       angelernten Nestern (ablageplatte_pose.xacro, tools/ablageplatte_modell.py). -->
+  <xacro:include filename="$(find mycobot_world)/urdf/ablageplatte.xacro"/>
+  <xacro:include filename="$(find mycobot_world)/urdf/ablageplatte_pose.xacro"/>
+  <!-- x-Position der vertikalen Säule (Kamera-Arm reicht von hier zur Kamera). -->
+  <xacro:property name="column_x" value="0.385"/>
   <!-- Haupt-Referenzframe (Master-Plan vorgeschrieben) +
        physisches Basis-Gehäuse des Roboters (Box mit USB/HMI-Anschluss, zwischen Arm und Boden).
        ~15×11×11 cm, auf Armachse zentriert, sitzt auf der Plattform (z=0) auf → z=0..0.11.
        HINZUGEFUEGT 2026-06-15: zuvor war robot_base ein leeres Link → Gehäuse fehlte im
-       Kollisionsmodell → bei sehr naher Schraube faltet sich der Arm und stößt an dieses
+       Kollisionsmodell → bei sehr naher Welle faltet sich der Arm und stößt an dieses
        Gehäuse, MoveIt sah es nicht. Nur-Kollision (Visual ist bereits im joint1-Mesh). -->
+  <!-- ✅ 2026-09-11 NACHGEMESSEN (Benutzer): 11 cm in x, 15 cm in y, 11 cm hoch.
+       Vorher stand hier 0.15 x 0.11 - die Achsen waren VERTAUSCHT. -->
   <link name="robot_base">
     <collision>
       <origin xyz="0 0 0.055" rpy="0 0 0"/>
-      <geometry><box size="0.15 0.11 0.11"/></geometry>
+      <geometry><box size="0.11 0.15 0.11"/></geometry>
     </collision>
   </link>
@@ -52,5 +71,5 @@
   <!--
     Kaiser RS 2 XA Repro-Stand (Baseboard ist platform_top oben).
-    Drei Teile: Halte-Klemme (tutucu_kelepce), vertikale Säule (column),
+    Drei Teile: Halte-Klemme (halteklemme), vertikale Säule (column),
     von column zum Roboter reichender horizontaler Kamera-Arm (camera_arm).
     Geometrie (robot_base frame):
@@ -61,5 +80,5 @@
         column+Klemme ~5cm näher an Roboter gebracht, sodass der Stab an beide Enden anschließt.
   -->
-  <link name="tutucu_kelepce">
+  <link name="halteklemme">
     <visual>
       <origin xyz="0 0 0" rpy="0 0 0"/>
@@ -74,7 +93,7 @@
     </collision>
   </link>
-  <joint name="robot_base_to_tutucu_kelepce" type="fixed">
+  <joint name="robot_base_to_halteklemme" type="fixed">
     <parent link="robot_base"/>
-    <child  link="tutucu_kelepce"/>
+    <child  link="halteklemme"/>
     <!-- 2026-06-25: zur Mitte der fernen Kante der Platte zurückgesetzt (0.3225 -> 0.3725).
          Die vorherige Position vom 2026-06-07 hatte den Stab ~5cm vor die Plattenkante verschoben. -->
@@ -101,10 +120,10 @@
          (Das vorherige 0.335 hatte den Stab ~5cm vor die Kante verschoben; der Kamera-Arm
          war deshalb auf 12.5cm verkürzt worden — jetzt ist der Arm wieder verlängert.) -->
-    <origin xyz="0.385 -0.125 0.38" rpy="0 0 0"/>
+    <origin xyz="${column_x} -0.125 0.38" rpy="0 0 0"/>
   </joint>
   <link name="camera_arm">
     <visual>
       <origin xyz="0 0 0" rpy="0 0 0"/>
-      <geometry><box size="0.229 0.025 0.025"/></geometry>
+      <geometry><box size="${column_x - cam_x} 0.025 0.025"/></geometry>
       <material name="arm_color">
         <color rgba="0.20 0.20 0.25 0.85"/>
@@ -113,5 +132,5 @@
     <collision>
       <origin xyz="0 0 0" rpy="0 0 0"/>
-      <geometry><box size="0.229 0.025 0.025"/></geometry>
+      <geometry><box size="${column_x - cam_x} 0.025 0.025"/></geometry>
     </collision>
   </link>
@@ -129,6 +148,160 @@
          berührt bei 0.385 die column. Länge=0.385-0.156=0.229. Mitte=(0.156+0.385)/2=0.2705.
          column (0->0.76m) ist hoch genug, unverändert. -->
-    <origin xyz="0.2705 -0.125 0.450" rpy="0 0 0"/>
-  </joint>
+    <origin xyz="${(cam_x + column_x) / 2} -0.125 ${cam_z}" rpy="0 0 0"/>
+  </joint>
+  <!--
+    ===================== BEREITSTELLUNGSSCHALE =====================
+    Kreisringausschnitt, am Bauteil gemessen (2026-09-09):
+      Bogenwinkel 45.3 Grad | R 186.9 .. 301.9 mm | Wand 2 mm | Wandhoehe 17 mm
+      (Winkel 2026-09-12 mit der Kamera an der OBERKANTE gemessen: 45.3 Grad, 5 Frames,
+       Spannweite 0.2 Grad, Radien bestaetigt; die 39.9 Grad aus 130/210/115 mm Lineal
+       gehoeren wohl zum Innenboden - die Silhouette ist oben rund 148/239 mm.
+       Fuer die Kollision zaehlt die Oberkante.)
+    Aufbau und Begruendung der Zerlegung stehen im Kopf von schale.xacro,
+    die Lage in schale_pose.xacro.
+    Sie steht standardmaessig NICHT im Modell: die Lage ist noch nicht gemessen,
+    und eine Schale an der falschen Stelle verwirft gueltige Griffe stillschweigend.
+    Nach `tools/schale_pose_klicken.py` mit SCHALE_MONTIERT=1 einschalten.
+  -->
+  <xacro:arg name="schale_montiert" default="false"/>
+  <xacro:arg name="schale_boden"    default="false"/>
+  <xacro:property name="schale_r_innen"  value="0.1869"/>   <!-- Innenflaeche der inneren Wand -->
+  <xacro:property name="schale_r_aussen" value="0.3019"/>   <!-- Aussenflaeche der aeusseren Wand -->
+  <xacro:property name="schale_winkel"   value="${45.3 * PI / 180.0}"/>   <!-- Oberkante, Kamera 2026-09-12 (vorher 39.9 aus Lineal) -->
+  <xacro:property name="schale_wand"     value="0.002"/>    <!-- gemessen 2026-09-09 -->
+  <xacro:property name="schale_hoehe"    value="0.017"/>    <!-- gemessen 2026-09-09, Innenboden bis Oberkante -->
+  <xacro:property name="schale_boden_dicke" value="0.002"/> <!-- ANNAHME = Wandstaerke, nicht gemessen -->
+  <xacro:property name="schale_segmente" value="6"/>        <!-- Sehnen-Kaesten je Bogen, Fehler 0.51 mm -->
+  <xacro:if value="$(arg schale_montiert)">
+    <!-- 2026-09-14: Waende als STL-Mesh mit RUNDEN Kanten (Benutzer: keine eckigen Ecken - oben, unten, innen,
+         aussen); erzeugt von tools/schale_mesh.py (Ecken r 10 mm, Wandprofil oben/unten halbrund) aus denselben
+         Massen. schale_mesh:=false -> alte Sehnen-Kaesten. -->
+    <xacro:arg name="schale_mesh" default="true"/>
+    <link name="schale">
+      <xacro:if value="$(arg schale_mesh)">
+        <visual>
+          <geometry><mesh filename="package://mycobot_world/meshes/schale_wand.stl"/></geometry>
+          <material name="schale_wand_farbe"><color rgba="0.75 0.70 0.55 0.45"/></material>
+        </visual>
+        <collision>
+          <geometry><mesh filename="package://mycobot_world/meshes/schale_wand.stl"/></geometry>
+        </collision>
+        <visual>
+          <geometry><mesh filename="package://mycobot_world/meshes/schale_boden.stl"/></geometry>
+          <material name="schale_boden_farbe_mesh"><color rgba="0.55 0.62 0.75 0.9"/></material>
+        </visual>
+        <xacro:if value="$(arg schale_boden)">
+          <collision><geometry><mesh filename="package://mycobot_world/meshes/schale_boden.stl"/></geometry></collision>
+        </xacro:if>
+      </xacro:if>
+      <xacro:unless value="$(arg schale_mesh)">
+        <xacro:schale_ringausschnitt r_innen="${schale_r_innen}" r_aussen="${schale_r_aussen}"
+                                     winkel="${schale_winkel}" wand="${schale_wand}"
+                                     hoehe="${schale_hoehe}" segmente="${schale_segmente}"
+                                     mit_boden="$(arg schale_boden)" boden="${schale_boden_dicke}"/>
+      </xacro:unless>
+    </link>
+    <joint name="robot_base_to_schale" type="fixed">
+      <parent link="robot_base"/>
+      <child  link="schale"/>
+      <origin xyz="${schale_x} ${schale_y} ${schale_z}" rpy="0 0 ${schale_yaw}"/>
+    </joint>
+  </xacro:if>
+  <!--
+    ===================== ABLAGEPLATTE (5 x 4 Nester) =====================
+    Festgeklebt seit 2026-09-11 (vier Ecknester angelernt, 16 gerechnet). Standard AN.
+    Lage/Bosse aus den angelernten Nestern (Modellraum), Masse real - s. ablageplatte.xacro.
+    Abschalten: ABLAGEPLATTE_MONTIERT=0 (z.B. wenn die Platte zum Anlernen weggenommen ist).
+  -->
+  <xacro:arg name="ablageplatte_montiert" default="true"/>
+  <xacro:if value="$(arg ablageplatte_montiert)">
+    <link name="ablageplatte">
+      <xacro:ablageplatte_koerper laenge_x="${ablageplatte_laenge_x}" laenge_y="${ablageplatte_laenge_y}"/>
+    </link>
+    <xacro:ablageplatte_boss_links/>   <!-- farbige Bosse als eigene Links (nur visual) -->
+    <joint name="robot_base_to_ablageplatte" type="fixed">
+      <parent link="robot_base"/>
+      <child  link="ablageplatte"/>
+      <origin xyz="${ablageplatte_x} ${ablageplatte_y} ${ablageplatte_z}" rpy="0 0 ${ablageplatte_yaw}"/>
+    </joint>
+  </xacro:if>
+  <!--
+    ===================== TRICHTER (Vereinzelung) =====================
+    Auslaufrohr Ø 17 / 20 mm hoch, schraege KEGELSCHALE (nur ein ~90-Grad-Bogen,
+    auf der dem Roboter abgewandten Seite) bis "Ø 85" in 95 mm, Fussplatte Ø 120. Am Bauteil gemessen 2026-09-10 (messungen_trichter.txt);
+    Aufbau, Annahmen und Zerlegungsfehler stehen im Kopf von trichter.xacro,
+    die Lage in trichter_pose.xacro.
+    Er steht standardmaessig NICHT im Modell: die Neigungsrichtung (yaw) ist noch
+    nicht gemessen. Nach dem Messen mit TRICHTER_MONTIERT=1 einschalten - und
+    VOR jeder Fahrt in Trichternaehe: am 2026-09-10 hat sich der Greifer dort
+    verbogen, weil der Trichter im Modell fehlte.
+  -->
+  <xacro:arg name="trichter_montiert" default="false"/>
+  <xacro:property name="trichter_auslauf_r_aussen" value="0.0075"/>  <!-- Ø 15 aussen (Benutzer 2026-09-12; vorher 17) -->
+  <!-- Auslaufrohr: Wand 5 mm -> Bohrung Ø 5 (Benutzer 2026-09-12). Im Kollisionsmodell bleibt
+       das Rohr VOLL (ein Zylinder) - in die Bohrung faehrt nichts ausser der Welle. Nur Notiz. -->
+  <xacro:property name="trichter_auslauf_wand"     value="0.005"/>
+  <xacro:property name="trichter_auslauf_hoehe"    value="0.020"/>   <!-- Auslaufkante ueber Grund, gemessen -->
+  <!-- ✅ 2026-09-12 GEMESSEN (Benutzer, rechtwinkliges Dreieck ab OBERKANTE des Auslaufrohrs):
+       Ankathete 40 mm (waagerecht), Gegenkathete 95 mm (senkrecht), Hypotenuse ~100 (103) mm
+       -> Wand 22.8 Grad aus der Senkrechten, Oberkante 20 + 95 = 115 mm ueber Grund,
+       40 mm weiter aussen als die Rohrkante. Der Kragen (Ø 15 -> 30 auf 17 mm = 23.8 Grad)
+       liegt auf DERSELBEN Flanke - die Wand ist ab der Rohrkante eine gerade schraege Flaeche. -->
+  <xacro:property name="trichter_kegel_hoehe"      value="0.095"/>   <!-- Rohrkante (20) bis Muendung (115) -->
+  <xacro:property name="trichter_kegel_r_oben"     value="0.0475"/>  <!-- Rohrkante 7.5 + 40 mm (Dreieck 2026-09-12) -->
+  <xacro:property name="trichter_wand"             value="0.002"/>   <!-- gemessen (17-13)/2 -->
+  <!-- Achsneigung: Standard = halber Oeffnungswinkel -> nahe Wand senkrecht (Linealprobe).
+       atan((42.5 - 6.5) / 75) = 25.6 Grad. ANNAHME, siehe Kopf von trichter.xacro. -->
+  <!-- Kragen auf der Auslaufkante (Benutzer 2026-09-12): Ø 30 aussen, 17 mm hoch, Wand 1 mm (bestaetigt) -->
+  <xacro:property name="trichter_kragen_r"         value="0.015"/>
+  <xacro:property name="trichter_kragen_hoehe"     value="0.017"/>
+  <xacro:property name="trichter_kragen_wand"      value="0.002"/>   <!-- Wand 2 mm wie die ganze Flanke (Benutzer 2026-09-12) -->
+  <xacro:property name="trichter_wand2_hoehe"      value="0.020"/>   <!-- robotseitige Wand: nur 20 mm ab Auslaufkante (2026-09-12) -->
+  <xacro:property name="trichter_wand2_wand"       value="0.001"/>   <!-- robotseitige Wand: 1 mm dick (hohe Wand 2 mm) -->
+  <!-- 2026-09-12: KEINE Achsneigung mehr - jede Wand ist ein Kegelsegment um die Rohrachse,
+       die Schraege steckt allein im Radiuszuwachs (7.5 -> 47.5 auf 95 mm = 22.8 Grad). -->
+  <xacro:property name="trichter_neigung"          value="0.0"/>
+  <!-- Kegelfuss liegt HINTER dem Auslaufrohr (Foto 15.18.54): Rohr-Aussenradius +
+       Kegelfuss-Radius = 8.5 + 8.5. ANNAHME tangential; siehe Kopf von trichter.xacro. -->
+  <xacro:property name="trichter_kegel_versatz"    value="0.017"/>
+  <!-- Der Kegel ist eine SCHALE (Benutzer 2026-09-11: "1/6 des Umfangs"), auf der
+       dem Roboter abgewandten Seite = Neigungsrichtung +X. Benutzer korrigiert auf "1/4" = 90 Grad (vorher 1/6), bis
+       Sehne + Pfeilhoehe der Muendung gemessen sind. Siehe Kopf von trichter.xacro. -->
+  <xacro:property name="trichter_kegel_bogen"      value="${90.0 * PI / 180.0}"/>
+  <xacro:property name="trichter_scheiben"         value="15"/>      <!-- 5 mm je Scheibe, Fehler 2.3 mm nach innen -->
+  <xacro:property name="trichter_sehnen"           value="4"/>       <!-- 22.5 Grad je Sehne, Fehler 0.8 mm -->
+  <xacro:property name="trichter_fuss_r"           value="0.045"/>   <!-- Ø 90 VORLAEUFIG (14.9.: Ø 120 ragte 19 mm zu weit zur Platte; Ecken real oval) -->
+  <xacro:property name="trichter_fuss_dicke"       value="0.004"/>   <!-- ANNAHME -->
+  <!-- 2026-09-12 (Benutzer): Fussplatte ist ein HALBKREIS; die gerade Kante liegt an der
+       robotseitigen Aussenkante des Auslaufrohrs, der Halbkreis reicht nach +X. -->
+  <xacro:property name="trichter_fuss_kante_x"     value="${-trichter_auslauf_r_aussen}"/>
+  <xacro:property name="trichter_zunge_laenge"     value="0.025"/>   <!-- ANNAHME -->
+  <xacro:property name="trichter_zunge_breite"     value="0.015"/>   <!-- ANNAHME -->
+  <xacro:property name="trichter_zunge_hoehe"      value="0.020"/>   <!-- ANNAHME: bis Auslaufkante -->
+  <xacro:if value="$(arg trichter_montiert)">
+    <link name="trichter">
+      <xacro:trichter_koerper auslauf_r_aussen="${trichter_auslauf_r_aussen}"
+                              auslauf_hoehe="${trichter_auslauf_hoehe}"
+                              kegel_hoehe="${trichter_kegel_hoehe}"
+                              kegel_r_oben="${trichter_kegel_r_oben}"
+                              wand="${trichter_wand}" neigung="${trichter_neigung}"
+                              kegel_versatz="${trichter_kegel_versatz}"
+                              kegel_bogen="${trichter_kegel_bogen}"
+                              scheiben="${trichter_scheiben}" sehnen="${trichter_sehnen}"
+                              fuss_r="${trichter_fuss_r}" fuss_dicke="${trichter_fuss_dicke}"
+                              fuss_kante_x="${trichter_fuss_kante_x}"
+                              zunge_laenge="${trichter_zunge_laenge}"
+                              zunge_breite="${trichter_zunge_breite}"
+                              zunge_hoehe="${trichter_zunge_hoehe}"
+                              kragen_r="${trichter_kragen_r}" kragen_hoehe="${trichter_kragen_hoehe}"
+                              kragen_wand="${trichter_kragen_wand}" wand2_hoehe="${trichter_wand2_hoehe}"
+                              wand2_wand="${trichter_wand2_wand}" auslauf_wand="${trichter_auslauf_wand}"/>
+    </link>
+    <joint name="robot_base_to_trichter" type="fixed">
+      <parent link="robot_base"/>
+      <child  link="trichter"/>
+      <origin xyz="${trichter_x} ${trichter_y} ${trichter_z}" rpy="0 0 ${trichter_yaw}"/>
+    </joint>
+  </xacro:if>
   <!-- mycobot-Arm + adaptive gripper: upstream-URDF-Inhalt -->
   <xacro:include filename="$(find mycobot_description)/urdf/mycobot_280_jn/mycobot_280_jn_adaptive_gripper.urdf"/>
@@ -140,14 +313,374 @@
   </joint>
   <!--
-    TCP (Tool Center Point) — Mittelpunkt zwischen den beiden Greifer-Fingern.
-    Pose etwa 9 cm voraus in z-Achsen-Richtung von gripper_base.
-    Master-Plan: Pick/Place-Bewegungen werden vom tcp-Frame aus gesteuert.
-  -->
+    ===================== GREIFERFINGER UND TCP =====================
+    Am 2026-09-09 wurden laengere Finger montiert. Der Nutzer hat nachgemessen:
+    vom Flansch bis zur Fingerspitze sind es jetzt 135 mm statt 110 mm.
+    Das passt genau: gripper_base sitzt im selben Ursprung wie joint6_flange
+    (das Gelenk joint6output_to_gripper_base hat origin "0 0 0"), die 110 mm
+    wurden also schon immer ab Flansch gerechnet. Die Finger sind um 25 mm
+    laenger geworden, also wandert die Spitze von 110 auf 135 mm.
+    Fingermass laut Nutzer (2026-09-09):
+      Laenge gesamt 50 mm; die ersten 25 mm durchgehend 20 mm breit,
+      die letzten 25 mm verjuengen sich von 20 mm auf 1 mm an der Spitze.
+      Vorher: 25 mm lang, 20 mm breit.
+    Daraus folgt: die Finger beginnen bei y = 135 - 50 = 85 mm.
+    WARUM DAS MODELLIERT WERDEN MUSS: bis hierher endete die gesamte
+    Greifergeometrie des Modells bei y ~ 42 mm (die Kollisionsbox von
+    gripper_base). Zwischen 42 mm und der Spitze bei 135 mm stand im Modell
+    NICHTS - weder sichtbar noch fuer die Kollisionspruefung. MoveIt konnte
+    also nicht sehen, wenn die Fingerspitzen in die Schale fahren. Mit den
+    25 mm laengeren Fingern ist genau das die Gefahr.
+    ⚠️ FOLGE FUER GRASP_Z_OFFSET: Der Wert -0.025 in run_pick_preview.sh ist
+    exakt so gross wie die Verlaengerung. Er hat sehr wahrscheinlich genau
+    diesen Modellfehler ausgeglichen (das Modell hielt die Spitze fuer 25 mm
+    zu weit oben, also musste der Griff 25 mm tiefer). Mit dem richtigen TCP
+    sollte er auf 0 gehen - ERST MESSEN, nicht blind beides aendern.
+    ANNAHME, die noch zu pruefen ist: die Dicke des Fingerblechs ist mit 6 mm
+    angesetzt (nicht gemessen), und die 20 mm Breite liegt quer zur
+    Schliessrichtung. In RViz gegen den echten Greifer vergleichen.
+    ================================================================
+  -->
+  <!-- ⚠️ 2026-09-11 KORRIGIERT, -34 mm. Die 135 mm sind vom FLANSCH bis zur
+       Fingerspitze gemessen (2026-09-09). Diese Masse zaehlen aber ab dem
+       Ursprung von gripper_base, und der liegt NICHT am Flansch: das Upstream-
+       URDF setzt joint6_flange -> gripper_base auf xyz 0 0 0.034 (die Notiz vom
+       2026-09-09 "gleicher Ursprung" hatte die auskommentierte Zeile gelesen).
+       Also Spitze = 135 - 34 = 101 mm ab gripper_base. Am Aufbau bestaetigt:
+       am Greifpunkt (Modell-TCP z 8.2) mass der Benutzer die Fingerspitze
+       40-42 mm ueber der Grundplatte, 1 mm unter der Kopfoberkante der Welle
+       -> 33 mm Fehler, das ist der Flanschversatz. Dieselben 34 mm erklaeren
+       den alten GRASP_Z_OFFSET -0.025 (TCP 110 mit den alten Fingern war um
+       denselben Betrag zu lang). -->
+  <xacro:property name="flansch_versatz" value="0.034"/>  <!-- joint6_flange -> gripper_base, Upstream -->
+  <xacro:property name="finger_start"  value="${0.085 - flansch_versatz}"/>   <!-- ab gripper_base: 51 mm -->
+  <xacro:property name="finger_tip"    value="${0.135 - flansch_versatz}"/>   <!-- ab gripper_base: 101 mm (Flansch->Spitze 135 gemessen) -->
+  <!-- ✅ 2026-09-11 NACHGEMESSEN (Benutzer): Finger 50 mm lang, in Schliessrichtung
+       15 mm (nicht 20); ab der Haelfte laeuft er dreieckig auf die Spitze zu.
+       Der Keil ist ein echtes Dreiecksprisma (STL), Innenflaeche eben, Spitze scharf. -->
+  <xacro:property name="finger_breit"  value="0.015"/>   <!-- gemessen: gerader Teil, 15 mm -->
+  <!-- Keil-Masse (15 x 25 x finger_tief) stecken im STL; bei Aenderung neu erzeugen (DEVLOG 2026-09-11). -->
+  <xacro:property name="finger_tief"   value="0.020"/>   <!-- ANNAHME aus den Fotos, nicht gemessen: Plattentiefe -->
+  <!-- Wie weit die INNENFLAECHE des Fingers von der Mittellinie weg ist.
+       Die Finger sitzen NICHT auf dem Ursprung von gripper_left1/right1 - der
+       ist der Drehpunkt des Traegers, nicht die Platte. Auf dem Foto der
+       geschlossenen Finger beruehren sich die Innenflaechen in der Mitte.
+       Beim ersten Versuch standen die Finger deshalb 78 mm auseinander und
+       schwebten an den Aussenkanten des Greifers.
+       ⚠️ 2026-09-11 KORRIGIERT. Vorher stand hier traeger_x = 39 mm - das ist
+       der Traegerursprung bei GELENKWERT 0. Gelenkwert 0 ist aber NICHT
+       "geschlossen": der Bereich ist [-0.74 zu .. +0.15 auf], 0 liegt bei 83 %
+       auf. Folge im alten Modell: Finger bei "auf" (0.15) nur 6 mm auseinander,
+       bei "zu" (-0.62) 26 mm ineinander. Damit stiess der OFFENE Greifer im
+       Modell mitten in das Auslaufrohr des Trichters (trichter_lage_pruefen.py:
+       Kontakt der Fingerspitze bei dx -3, dy -4 - der Wellenachse).
+       Per FK (Sim-Stack, gripper_base-Frame) steht der Traeger bei:
+           +0.15 (auf)   x = +-41.1 mm
+            0.00         x = +-39.0
+           -0.62 (Griff) x = +-24.7
+           -0.74 (zu)    x = +-21.2   <- hier beruehren sich die Innenflaechen
+       Also: Innenflaeche = Traeger-x bei -0.74 minus finger_innen. Damit oeffnet
+       das Modell auf 42 mm; aus der Messung 6.8 mm bei 21 % folgen linear rund
+       32 mm - die Upstream-Kinematik ueberzeichnet den Hub also um ~5 mm je
+       Seite, mit dem Messschieber bei 100 % nachmessen. Bei -0.62 stehen die
+       Modellfinger 7 mm auseinander, die Firmware sagt 13 % ~ 4 mm. -->
+  <xacro:property name="finger_innen"  value="0.001"/>   <!-- Innenflaeche 1 mm neben der Mitte (geschlossen) -->
+  <xacro:property name="traeger_x"     value="0.0212"/>  <!-- Traeger-x bei GESCHLOSSEN (-0.74), per FK -->
+  <xacro:property name="finger_z"      value="-0.01"/>   <!-- gleiche Hoehe wie der tcp -->
+  <xacro:property name="gummi_dicke"   value="0.003"/>   <!-- Reibgummi an der Spitze, gemessen 2026-09-11 -->
+  <xacro:property name="gummi_kante"   value="0.013"/>   <!-- 13 x 13 mm -->
+  <!-- Ein Finger als zwei Quader: gerades Stueck + verjuengte Spitze.
+       seite = "links" oder "rechts"; x_link = x-Lage des tragenden Link im
+       gripper_base (die Finger sitzen bei -0.039 bzw. +0.039). -->
+  <xacro:macro name="greiferfinger" params="name parent x_link innen">
+    <link name="${name}">
+      <!-- Gerades Stueck (erste 25 mm): volle 15 mm in Schliessrichtung (x). -->
+      <visual>
+        <geometry>
+          <box size="${finger_breit} ${0.025} ${finger_tief}"/>
+        </geometry>
+        <origin xyz="${innen * (traeger_x - finger_innen - finger_breit/2)} ${finger_start + 0.0125 - 0.021} ${finger_z}" rpy="0 0 0"/>
+        <material name="finger_weiss"><color rgba="0.92 0.92 0.90 1.0"/></material>
+      </visual>
+      <!-- Keil (letzte 25 mm): echtes Dreiecksprisma als STL (meshes/finger_keil_*.stl,
+           Meter, erzeugt 2026-09-11): Innenflaeche eben, Aussenkante laeuft auf die
+           SPITZE zu. _neg = Koerper zu -x (linker Finger), _pos = zu +x (rechter).
+           Ursprung des Mesh = Innenflaeche am Keilfuss, z-mittig. -->
+      <xacro:property name="keil_datei" value="package://mycobot_world/meshes/finger_keil_${'neg' if innen > 0 else 'pos'}.stl"/>
+      <visual>
+        <geometry><mesh filename="${keil_datei}"/></geometry>
+        <origin xyz="${innen * (traeger_x - finger_innen)} ${finger_start + 0.025 - 0.021} ${finger_z}" rpy="0 0 0"/>
+        <material name="finger_weiss"><color rgba="0.92 0.92 0.90 1.0"/></material>
+      </visual>
+      <collision>
+        <geometry><mesh filename="${keil_datei}"/></geometry>
+        <origin xyz="${innen * (traeger_x - finger_innen)} ${finger_start + 0.025 - 0.021} ${finger_z}" rpy="0 0 0"/>
+      </collision>
+      <!-- ✅ 2026-09-11 Reibgummi (Benutzer): 13 x 13 mm, 3 mm dick, auf der
+           INNENFLAECHE an der Fingerspitze (untere Kante), links und rechts.
+           Die Innenflaeche liegt damit 3 mm naeher an der Mitte; ganz zu (-0.74)
+           ueberlappen die Gummis im Modell (Paar finger_links/rechts ist im SRDF
+           ausgeschaltet) - physisch stoppt der Greifer frueher, die Firmware
+           meldet trotzdem den KOMMANDIERTEN Wert (0 %). -->
+      <visual>
+        <geometry><box size="${gummi_dicke} ${gummi_kante} ${gummi_kante}"/></geometry>
+        <origin xyz="${innen * (traeger_x - finger_innen + gummi_dicke/2)} ${finger_tip - 0.021 - gummi_kante/2} ${finger_z}" rpy="0 0 0"/>
+        <material name="gummi_schwarz"><color rgba="0.15 0.15 0.15 1.0"/></material>
+      </visual>
+      <collision>
+        <geometry><box size="${gummi_dicke} ${gummi_kante} ${gummi_kante}"/></geometry>
+        <origin xyz="${innen * (traeger_x - finger_innen + gummi_dicke/2)} ${finger_tip - 0.021 - gummi_kante/2} ${finger_z}" rpy="0 0 0"/>
+      </collision>
+    </link>
+    <joint name="${parent}_to_${name}" type="fixed">
+      <parent link="${parent}"/>
+      <child  link="${name}"/>
+      <origin xyz="0 0 0" rpy="0 0 0"/>
+    </joint>
+  </xacro:macro>
+  <!-- Die Finger haengen an gripper_left1/right1, den aeussersten beweglichen
+       Gliedern; sie machen das Oeffnen und Schliessen also mit. -->
+  <xacro:greiferfinger name="finger_links"  parent="gripper_left1"  x_link="-0.039" innen="1"/>
+  <xacro:greiferfinger name="finger_rechts" parent="gripper_right1" x_link="0.039" innen="-1"/>
+  <!--
+    Oberseite des Greifers: bis 2026-09-11 standen hier ein weisser Vorsprung
+    ("halter_sockel", ab Werk) und darauf ein schwarzes P-foermiges Halteteil fuer die
+    Elephant-Kamera ("kamerahalter"). ✅ 2026-09-11: der Benutzer hat BEIDE entfernt -
+    Links, Joints und SRDF-Paare sind gestrichen. Die Masse unten bleiben nur als Notiz,
+    falls etwas davon wieder drankommt. Oberseite des Greiferkoerpers = greifer_huelle.
+  -->
+  <xacro:property name="halter_breite" value="0.025"/>   <!-- weisser Vorsprung, x -->
+  <xacro:property name="halter_laenge" value="0.035"/>   <!-- weisser Vorsprung, y -->
+  <xacro:property name="halter_hoehe"  value="0.020"/>   <!-- weisser Vorsprung, z -->
+  <xacro:property name="halter_x"      value="0.0"/>     <!-- mittig -->
+  <xacro:property name="halter_y"      value="0.020"/>   <!-- 2 cm vor dem Flanschanschluss -->
+  <xacro:property name="koerper_oben"  value="0.01734"/> <!-- Oberseite Greiferkoerper -->
+  <xacro:property name="halter_z"      value="${koerper_oben + halter_hoehe/2}"/>
+  <!-- Steg des P: liegt auf dem weissen Vorsprung -->
+  <xacro:property name="steg_laenge"   value="0.039"/>
+  <xacro:property name="steg_breite"   value="0.020"/>
+  <xacro:property name="steg_dicke"    value="0.010"/>
+  <xacro:property name="steg_z"        value="${koerper_oben + halter_hoehe + steg_dicke/2}"/>
+  <!-- Kopf des P: neben dem Vorsprung, auf dessen Hoehe -->
+  <xacro:property name="kopf_laenge"   value="0.030"/>
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